File: throttle-tune/pcb_throttle-tune/throttle-tune.kicad_pcb (KiCad board)
At the start: 2 copper layers, 74.7 x 69.1 mm, 51 parts, among them IC1 ATMEGA8A-P, J1 3speedSw-in, J10 9V supply / small battery, J2 gas-pedal-in, J3 throttle-out, J4 3speedSw-out, J5 UART [TX, RX, GND], J7 gpio-reserve, J8 reserve, reverse-sw, J9 5V/GND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

Commit message: pcb: optimize text, comments, Add README
Parts:
- J1: value 3speedSw-in -> 3-speed-IN: COM, sw-fast, sw-slow
- J10: value 9V supply / small battery -> 9V supply batt: GND, 9V
- J2: value gas-pedal-in -> gas-pedal-IN: GND, Analog, 5V-motorctl
- J3: value throttle-out -> throttle-OUT: GND, Analog, 5V-motorctl
- J4: value 3speedSw-out -> 3-speed-OUT: COM, sw-fast, sw-slow
- J9: value 5V/GND -> 5V out, GND
Other:
- board text added: "dropped (motorcontroller not connected here)"
Changed lines of the file:
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@@
 			)
 		)
-		(property "Value" "9V supply / small battery"
-			(at 0.508 7.62 90)
+		(property "Value" "9V supply batt: GND, 9V"
+			(at 5.912 9.596 90)
 			(layer "F.Fab")
 			(effects
@@
 			)
 		)
-		(property "Value" "3speedSw-in"
-			(at 4.572 6.604 0)
+		(property "Value" "3-speed-IN: COM, sw-fast, sw-slow"
+			(at 7.564 6.604 0)
 			(layer "F.Fab")
 			(effects
@@
 		(tags "Resistor Axial_DIN0207 series Axial Horizontal pin pitch 10.16mm 0.25W = 1/4W length 6.3mm diameter 2.5mm")
 		(property "Reference" "R12"
-			(at 5.08 -2.37 360)
+			(at 5.08 -2.37 0)
 			(layer "F.SilkS")
 			(effects
@@
 		)
 		(property "Value" "47k"
-			(at 5.08 2.37 360)
+			(at 5.08 2.37 0)
 			(layer "F.Fab")
 			(effects
@@
 		)
 		(fp_text user "${REFERENCE}"
-			(at 5.08 0 360)
+			(at 5.08 0 0)
 			(layer "F.Fab")
 			(effects
@@
 		(tags "to-92 sc-43 sc-43a sot54 PA33 transistor")
 		(property "Reference" "Q2"
-			(at 2.54 -3.56 360)
+			(at 2.54 -3.56 0)
 			(layer "F.SilkS")
 			(effects
@@
 		)
 		(property "Value" "BC547"
-			(at 2.54 2.79 360)
+			(at 2.54 2.79 0)
 			(layer "F.Fab")
 			(hide yes)
@@
 		)
 		(property "Footprint" "Package_TO_SOT_THT_AKL:TO-92_Inline_Wide_CBE"
-			(at 0 0 360)
+			(at 0 0 0)
 			(layer "F.Fab")
 			(hide yes)
@@
 		)
 		(property "Datasheet" "https://www.tme.eu/Document/6c5d898a533a0762c2bc33eb26c283a8/BC546-550-DTE.pdf"
-			(at 0 0 360)
+			(at 0 0 0)
 			(layer "F.Fab")
 			(hide yes)
@@
 		)
 		(property "Description" "NPN TO-92 transistor, 45V, 100mA, 500mW, Complementary to BC557, Alternate KiCAD Library"
-			(at 0 0 360)
+			(at 0 0 0)
 			(layer "F.Fab")
 			(hide yes)
@@
 		)
 		(fp_text user "${REFERENCE}"
-			(at 2.54 0 360)
+			(at 2.54 0 0)
 			(layer "F.Fab")
 			(effects
@@
 			)
 		)
-		(property "Value" "gas-pedal-in"
-			(at 5.08 5.08 0)
+		(property "Value" "gas-pedal-IN: GND, Analog, 5V-motorctl"
+			(at 0.9 7.008 0)
 			(layer "F.Fab")
 			(effects
@@
 			)
 		)
-		(property "Value" "3speedSw-out"
-			(at 4.572 6.604 0)
+		(property "Value" "3-speed-OUT: COM, sw-fast, sw-slow"
+			(at 11.196 9.088 0)
 			(layer "F.Fab")
 			(effects
@@
 			)
 		)
-		(property "Value" "5V/GND"
-			(at 3.048 7.62 90)
+		(property "Value" "5V out, GND"
+			(at 2.672 7.596 90)
 			(layer "F.Fab")
 			(effects
@@
 		(tags "C Disc series Radial pin pitch 5.00mm  diameter 7mm width 2.5mm Capacitor")
 		(property "Reference" "C9"
-			(at 2.5 0 360)
+			(at 2.5 0 0)
 			(layer "F.SilkS")
 			(effects
@@
 		)
 		(property "Value" "100nF"
-			(at 4.024 -2.032 360)
+			(at 4.024 -2.032 0)
 			(layer "F.Fab")
 			(effects
@@
 		)
 		(fp_text user "${REFERENCE}"
-			(at 2.5 0 360)
+			(at 2.5 0 0)
 			(layer "F.Fab")
 			(effects
@@
 			)
 		)
-		(property "Value" "throttle-out"
-			(at 5.08 5.08 0)
+		(property "Value" "throttle-OUT: GND, Analog, 5V-motorctl"
+			(at -0.136 5.08 0)
 			(layer "F.Fab")
 			(effects
@@
 		)
 		(property "Value" "gpio-reserve"
-			(at 2.032 5.08 0)
+			(at 2.032 4.508 0)
 			(layer "F.Fab")
 			(effects
@@
 		)
 		(property "Value" "reserve, reverse-sw"
-			(at 6.096 5.08 0)
+			(at 4.96 7.008 0)
 			(layer "F.Fab")
 			(effects
@@
 		(layer "Edge.Cuts")
 	)
+	(gr_text "dropped\n(motorcontroller not connected here)"
+		(at 54 -3.5 0)
+		(layer "Dwgs.User")
+		(effects
+			(font
+				(size 1 1)
+				(thickness 0.15)
+			)
+			(justify left bottom)
+		)
+	)
 	(segment
